File: Power/12to5/12to5.sch (KiCad schematic (older format))
At the start: 9 parts

Commit message: Added PCB Added Gerbers Rev 1.0 Complete
Parts:
- gave numbers to parts that had none: 8
- renumbered +12V to CON1
Connections:
- net +5V: now also U1.2 (OUT), U1.4 (TAB)
Other:
- moved on the sheet: CON1, CON2, CON3, USB1
